File: mainboard/mainboard/mainboard.kicad_sch (KiCad schematic)
At the start: 1 part

Commit message: added gerber files
Parts:
- added M1: Motor_DC, Connector_PinHeader_1.27mm:PinHeader_1x02_P1.27mm_Vertical, symbol Motor:Motor_DC
- added Q1: P2N2222A, vision-empower:ON_Semi-CASE_2911-0-0-0, symbol vision-empower:P2N2222A
- added R1: 1k, Resistor_THT:R_Axial_DIN0207_L6.3mm_D2.5mm_P7.62mm_Horizontal, symbol Device:R
- added U1: LS_CONN, Connector_PinHeader_1.27mm:PinHeader_1x03_P1.27mm_Vertical, symbol vision-empower:LS_CONN
Connections:
- net at A1.22 (A3): now also U1.2 (SIG)
- net +5V: now reaches A1.27 (+5V)
- net +5V: now also M1.1 (+), U1.1 (VCC)
- net Earth: now reaches A1.29 (GND), A1.4 (GND)
- net Earth: now also Q1.3 (EMITTER), U1.3 (GND)
- net T1: now reaches A1.6 (D3)
- net T1: now also R1.1
- new net: Q1.2 (BASE), R1.2
- new net: M1.2 (-), Q1.1 (COLLECTOR)
